File: RF/bitx40_osc_pcb/bitx40_osc_pcb.sch (KiCad schematic (older format))
At the start: 16 parts, among them J1 Alim 5V, J2 Variable Capacitor, J3 Oscillator Output, Q1 2N3904, Q2 2N3904

Commit message: Correct 2N3904 package & review (ok)
Parts:
- removed Q1, Q2: 2N3904, Package_TO_SOT_THT:TO-92, symbol Device:Q_NPN_BEC
- added Q1, Q2: 2N3904, Package_TO_SOT_THT:TO-92, symbol Device:Q_NPN_CBE
Changed lines of the file:
@@
 EESchema Schematic File Version 4
+LIBS:bitx40_osc_pcb-cache
 EELAYER 26 0
 EELAYER END
@@
 $EndComp
 $Comp
-L Device:Q_NPN_BEC Q1
-U 1 1 5CCDF002
-P 3350 1550
-F 0 "Q1" H 3541 1596 50  0000 L CNN
-F 1 "2N3904" H 3541 1505 50  0000 L CNN
-F 2 "Package_TO_SOT_THT:TO-92" H 3550 1650 50  0001 C CNN
-F 3 "~" H 3350 1550 50  0001 C CNN
-	1    3350 1550
-	1    0    0    -1
-$EndComp
-$Comp
 L Device:R R4
 U 1 1 5CCDF4A3
@@
 F 3 "~" H 4300 1700 50  0001 C CNN
 	1    4300 1700
-	1    0    0    -1
-$EndComp
-$Comp
-L Device:Q_NPN_BEC Q2
-U 1 1 5CCDF5FB
-P 4750 1300
-F 0 "Q2" H 4941 1346 50  0000 L CNN
-F 1 "2N3904" H 4941 1255 50  0000 L CNN
-F 2 "Package_TO_SOT_THT:TO-92" H 4950 1400 50  0001 C CNN
-F 3 "~" H 4750 1300 50  0001 C CNN
-	1    4750 1300
 	1    0    0    -1
 $EndComp
@@
 Wire Wire Line
 	5650 1850 5650 2050
+$Comp
+L Device:Q_NPN_CBE Q1
+U 1 1 5CCEAE62
+P 3350 1550
+F 0 "Q1" H 3541 1596 50  0000 L CNN
+F 1 "2N3904" H 3541 1505 50  0000 L CNN
+F 2 "Package_TO_SOT_THT:TO-92" H 3550 1650 50  0001 C CNN
+F 3 "~" H 3350 1550 50  0001 C CNN
+	1    3350 1550
+	1    0    0    -1
+$EndComp
+$Comp
+L Device:Q_NPN_CBE Q2
+U 1 1 5CCEBB6C
+P 4750 1300
+F 0 "Q2" H 4941 1346 50  0000 L CNN
+F 1 "2N3904" H 4941 1255 50  0000 L CNN
+F 2 "Package_TO_SOT_THT:TO-92" H 4950 1400 50  0001 C CNN
+F 3 "~" H 4750 1300 50  0001 C CNN
+	1    4750 1300
+	1    0    0    -1
+$EndComp
 $EndSCHEMATC
